File: PCB design/self_balancing_robot.kicad_pcb (KiCad board)
At the start: 2 copper layers, 72.8 x 44.8 mm, 31 parts, among them J1 I2C, J2 Analog, J3 left_engine, J4 right_engine, J5 L293D_left, J6 SPI, J7 UART, J8 L293D_right, J9 input_supply, SW1 SW_Push, U1 ATmega328P-A, U4 LP2985-3.3, U5 NCP1117-5.0_SOT223, Y1 Crystal

Commit message: Update in PCB - almost finish version
Parts:
- removed J6: SPI, Connector_PinSocket_2.54mm:PinSocket_1x06_P2.54mm_Vertical
- added J10: SPI, Connector_PinSocket_2.54mm:PinSocket_1x07_P2.54mm_Vertical, F.Cu at (135.0, 117.0)
- moved C6 53.4 mm to (119.2, 99.1), turned to -90 degrees
- moved C7 48.8 mm to (119.2, 105.8), turned to 90 degrees
- moved Y1 47.6 mm to (115.0, 100.1), turned to -90 degrees
- moved J4 42.8 mm to (150.0, 79.0), turned to 180 degrees
- moved J7 40.3 mm to (103.2, 117.0)
- moved J3 36.3 mm to (146.5, 115.0)
- moved R5 31.3 mm to (93.5, 78.9)
- moved C5 30.4 mm to (96.4, 97.0), turned to -90 degrees
- moved C2 29.2 mm to (120.2, 93.5), turned to -90 degrees
- moved U1 28.8 mm to (129.0, 94.0)
- moved J1 28.6 mm to (90.9, 82.5)
- moved C3 28.4 mm to (136.5, 94.5), turned to -90 degrees
- moved C1 27.1 mm to (117.5, 93.5), turned to -90 degrees
- moved R4 26.3 mm to (96.0, 79.0)
- moved C14 25.4 mm to (114.2, 93.7), turned to -90 degrees
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Connections:
- J5 pad 1: PB1 -> PD6
- R3 pad 1: PD6 -> PB1
Routing:
- net +7.2V: track 3.88 -> 0.00 mm

Commit message: Cleaning in files part 1
Parts:
- removed J2: Analog, Connector_PinSocket_2.54mm:PinSocket_1x06_P2.54mm_Vertical
- moved J10 40.3 mm to (140.1, 77.0)
- moved J7 40.1 mm to (105.9, 77.0)
- moved D3 32.0 mm to (103.0, 110.0), turned to 0 degrees
- moved R3 27.5 mm to (107.8, 110.0), turned to 180 degrees
- moved J8 17.2 mm to (135.0, 90.5), turned to 90 degrees
- moved C4 14.1 mm to (89.5, 94.0), turned to 0 degrees
- moved C3 14.1 mm to (122.5, 93.5), turned to 180 degrees
- moved U1 13.8 mm to (115.2, 93.9)
- moved J5 13.7 mm to (134.9, 98.5), turned to 90 degrees
- moved C14 13.0 mm to (101.5, 91.0)
- moved C1 13.0 mm to (104.8, 91.0)
- moved C2 13.0 mm to (107.5, 91.0)
- moved U4 12.2 mm to (89.5, 90.5), turned to 90 degrees
- moved C5 12.1 mm to (89.5, 87.0), turned to 180 degrees
- moved Y1 12.0 mm to (103.5, 96.5)
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Connections:
- J10 pad 3: MISO -> MOSI
- J10 pad 4: MOSI -> MISO
- J4 pad 1: ENGINE_RIGHT_VCC -> ENGINE_RIGHT_GND
- J4 pad 2: ENGINE_RIGHT_GND -> ENGINE_RIGHT_VCC
Routing:
- net +5V: track 0.00 -> 138.8 mm, vias 0 -> 2
- net +7.2V: track 0.00 -> 72.0 mm
- net PD4: track 0.00 -> 55.0 mm, vias 0 -> 2
- net PD3: track 0.00 -> 42.1 mm, vias 0 -> 1
- net PD7: track 0.00 -> 40.3 mm, vias 0 -> 1
- net SCL_CONN: track 0.00 -> 34.8 mm, vias 0 -> 1
- net MOSI: track 0.00 -> 33.6 mm
- net CS: track 0.00 -> 33.3 mm, vias 0 -> 2
- net SDA_CONN: track 0.00 -> 32.9 mm, vias 0 -> 1
- net PD5: track 0.00 -> 32.6 mm, vias 0 -> 2
- net MISO: track 0.00 -> 29.6 mm
- net RESET_CONN: track 0.00 -> 29.3 mm, vias 0 -> 2
- net PD6: track 0.00 -> 27.6 mm, vias 0 -> 1
- net PD2: track 0.00 -> 27.3 mm, vias 0 -> 1
- net SCK: track 0.00 -> 25.9 mm
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